File: hardware/rtd-readout.kicad_sch (KiCad schematic)
At the start: 32 parts, among them J1 Conn_RTD_4W, J4 Conn_T7_RJ45, J5 Conn_T7_I2C, J6 Conn_Power, U1 ADS1115IDGS (0x48), U2 ADS1115IDGS (0x49)

Commit message: rev-G.1: J5 -> Molex PicoBlade 53048-0410 (no-crimp pre-made pigtail 2181120404)
Lucas found the 218112 PicoBlade pigtail family - swapped the I2C header
so the pre-made 425mm assembly plugs straight in (zero crimping). Pin
order (1=SCL..4=VS) unchanged; I2C re-routed as 4 parallel diagonals to
the new 1.25mm pads. Panel DXF, PANELS_AND_PINOUTS, BOM_REVIEW, order
CSV updated; DKRed zip regenerated.

Gates: ERC 0/0, DRC 0 violations / 0 unconnected.

Co-Authored-By: Claude Fable 5 <noreply@anthropic.com>
Parts:
- J5: footprint rtd-readout:Molex_KK-254_AE-7395-04A_1x04_P2.54mm_Horizontal -> rtd-readout:Molex_PicoBlade_53048-0410_1x04_P1.25mm_Horizontal; MPN 22-05-7048 -> 53048-0410; Manufacturer Molex (KK 254; mate: housing 22-01-3047 + crimps 0008500160) -> Molex (PicoBlade; mate: pre-made pigtail 2181120404, 425 mm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
Changed lines of the file:
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@@
 			)
 		)
-		(property "Footprint" "rtd-readout:Molex_KK-254_AE-7395-04A_1x04_P2.54mm_Horizontal"
+		(property "Footprint" "rtd-readout:Molex_PicoBlade_53048-0410_1x04_P1.25mm_Horizontal"
 			(at 298.45 53.34 0)
 			(show_name no)
@@
 			)
 		)
-		(property "MPN" "22-05-7048"
+		(property "MPN" "53048-0410"
 			(at 298.45 53.34 0)
 			(show_name no)
@@
 			)
 		)
-		(property "Manufacturer" "Molex (KK 254; mate: housing 22-01-3047 + crimps 0008500160)"
+		(property "Manufacturer" "Molex (PicoBlade; mate: pre-made pigtail 2181120404, 425 mm - NO crimping)"
 			(at 298.45 53.34 0)
 			(show_name no)
